Commit message: Added more detail to TB2 URDF file

File: turtlebot2_main/urdf/turtlebot2_se.urdf (robot description, URDF)
Before this commit: robot turtlebot2_astra, 3 links, 2 joints
Links:
- added link camera_depth_frame
- added link camera_depth_optical_frame
- added link front_caster_link, mass 0.03; collision sphere radius=0.018; visual sphere radius=0.018
- added link left_wheel_link, mass 0.08; collision cylinder length=0.018 radius=0.035; visual cylinder length=0.018 radius=0.035
- added link rear_caster_link, mass 0.03; collision sphere radius=0.018; visual sphere radius=0.018
- added link right_wheel_link, mass 0.08; collision cylinder length=0.018 radius=0.035; visual cylinder length=0.018 radius=0.035
- link base_link: mass None -> 2.4; geometry collision cylinder length=0.09 radius=0.178; visual cylinder length=0.09 radius=0.178
- link camera_link: mass None -> 0.15; geometry collision box size=0.045 0.165 0.045; visual box size=0.045 0.165 0.045
Joints:
- added joint camera_depth_joint: type fixed, parent camera_link, child camera_depth_frame, origin xyz=0 0 0
- added joint camera_depth_optical_joint: type fixed, parent camera_depth_frame, child camera_depth_optical_frame, origin xyz=0 0 0 rpy=-1.57079632679 0 -1.57079632679
- added joint front_caster_joint: type fixed, parent base_link, child front_caster_link, origin xyz=0.13 0 0
- added joint left_wheel_joint: type continuous, parent base_link, child left_wheel_link, origin xyz=0 0.145 0.035, axis 0 1 0
- added joint rear_caster_joint: type fixed, parent base_link, child rear_caster_link, origin xyz=-0.13 0 0
- added joint right_wheel_joint: type continuous, parent base_link, child right_wheel_link, origin xyz=0 -0.145 0.035, axis 0 1 0
- joint base_to_camera_joint: origin xyz=0.16 0 0.17 rpy=0 0 0 -> xyz=0.16 0 0.20
- joint footprint_to_base_joint: origin xyz=0 0 0.02 rpy=0 0 0 -> xyz=0 0 0
